Commit message: update codes.

File: tb3jp_description/robots/tb3jp_vegan.urdf.xacro (robot description, xacro)
@@ -175,49 +175,4 @@
     </inertial>
   </link>-->
-  <joint name="camera_joint" type="fixed">
-    <origin xyz="0.064 -0.065 0.094" rpy="0 0 0"/>
-    <parent link="base_link"/>
-    <child link="camera_link"/>
-  </joint>
-  <link name="camera_link">
-    <visual>
-     <origin xyz="0 0 0" rpy="${M_PI*0.5} 0 ${M_PI*0.5}"/>
-      <geometry>
-       <mesh filename="package://turtlebot3_description/meshes/sensors/r200.dae" />
-      </geometry>
-    </visual>
-    <collision>
-      <origin xyz="0.003 0.065 0.010" rpy="0 0 0"/>
-      <geometry>
-        <box size="0.008 0.130 0.022"/>
-      </geometry>
-    </collision>
-    <!-- This inertial field needs doesn't contain reliable data!! -->
-<!--   <inertial>
-      <mass value="0.564" />
-      <origin xyz="0 0 0" />
-      <inertia ixx="0.003881243" ixy="0.0" ixz="0.0"
-               iyy="0.000498940" iyz="0.0"
-               izz="0.003879257" />
-    </inertial>-->
-  </link>
-  <joint name="camera_rgb_joint" type="fixed">
-    <origin xyz="${r200_cam_rgb_px} ${r200_cam_rgb_py} ${r200_cam_rgb_pz}" rpy="0 0 0"/>
-    <parent link="camera_link"/>
-    <child link="camera_rgb_frame"/>
-  </joint>
-  <link name="camera_rgb_frame"/>
-  <joint name="camera_rgb_optical_joint" type="fixed">
-    <origin xyz="0 0 0" rpy="${-M_PI/2} 0 ${-M_PI/2}"/>
-    <parent link="camera_rgb_frame"/>
-    <child link="camera_rgb_optical_frame"/>
-  </joint>
-  <link name="camera_rgb_optical_frame"/>
-  <joint name="camera_depth_joint" type="fixed">
-    <origin xyz="${r200_cam_rgb_px} ${r200_cam_rgb_py + r200_cam_depth_offset} ${r200_cam_rgb_pz}" rpy="0 0 0"/>
-    <parent link="camera_link"/>
-    <child link="camera_depth_frame"/>
-  </joint>
-  <link name="camera_depth_frame"/>
   <!-- ZED use xacro include -->
 </robot>

File: tb3jp_description/urdf/sensors/zed.urdf.xacro (robot description, xacro)
@@ -56,5 +56,6 @@
       <parent link="zed_center"/>
       <child link="zed_left_camera"/>
-      <origin xyz="0 0.06 0" rpy="0 0 0" />
+      <origin xyz="0 0.06 0" rpy="-1.5707963267948966 0 -1.5707963267948966" />
+      <!-- <origin xyz="0 0.06 0" rpy="0 0 0" /> -->
     </joint>
     <joint name="zed_depth_camera_joint" type="fixed">
